Commit message: Add ADS device-notification read path (default)
Replace the per-cycle synchronous SUM read with PLC-pushed ADS device
notifications cached in lock-free slots, so read() does no network I/O and
the control loop is decoupled from network latency. Now the default;
read_mode=polling restores the synchronous SUM read. Write path unchanged.

- Per-symbol notification registered by symbol name via AdsNotification RAII
- Background callback decodes samples into atomic<double> cache (acquire/release)
- Process-static context registry indexed by uint32 hUser (no 64-bit ptr in hUser)
- Context published before registration (callback can fire from the ctor)
- Notifications torn down before AdsDevice (deleter dereferences the device)
- Per-interface URDF tuning: notify_mode (onchange/cyclic), notify_cycle_ms,
  notify_max_delay_ms (ms -> 100ns ticks)
- Shared decode_plc_element helper for both read paths
- Element offsets keyed by URDF index (mirrors SUM-read), not dense 0..n-1
- Demo: currentPos streamed cyclically at 1ms; fix MAIN.motionType state
  type USINT to match the PLC/command (was UDINT)

File: beckhoff_ads_bringup/urdf/beckhoff_bot/beckhoff_ads_interfaces.ros2_control.xacro (robot description, xacro)
@@ -14,5 +14,5 @@
         </command_interface>
     </xacro:macro>
-    <xacro:macro name="state_interface_PLC" params="name PLC_symbol PLC_type n_elements:=1 index:=''">
+    <xacro:macro name="state_interface_PLC" params="name PLC_symbol PLC_type n_elements:=1 index:='' notify_mode:='' notify_cycle_ms:='' notify_max_delay_ms:=''">
         <state_interface name="${name}">
             <param name="PLC_symbol">${PLC_symbol}</param>
@@ -22,4 +22,17 @@
                 <param name="index">${index}</param>
             </xacro:if>
+            <!-- Notification tuning (used when the hardware runs read_mode=notification).
+                 notify_mode: onchange (default) | cyclic. notify_cycle_ms / notify_max_delay_ms
+                 are milliseconds. One notification covers the whole symbol; the first interface
+                 naming a symbol sets its config. -->
+            <xacro:if value="${notify_mode != ''}">
+                <param name="notify_mode">${notify_mode}</param>
+            </xacro:if>
+            <xacro:if value="${notify_cycle_ms != ''}">
+                <param name="notify_cycle_ms">${notify_cycle_ms}</param>
+            </xacro:if>
+            <xacro:if value="${notify_max_delay_ms != ''}">
+                <param name="notify_max_delay_ms">${notify_max_delay_ms}</param>
+            </xacro:if>
         </state_interface>
     </xacro:macro>

File: beckhoff_ads_bringup/urdf/beckhoff_bot/beckhoff_bot_macro.ros2_control.xacro (robot description, xacro)
@@ -5,5 +5,6 @@
                 name
                 mock_hardware:=false
-                mock_sensor_commands:=false"
+                mock_sensor_commands:=false
+                read_mode:=notification"
                 >
         <ros2_control name="${name}" type="system">
@@ -19,4 +20,6 @@
                 <param name="plc_ams_port">851</param>
                 <param name="local_ams_net_id">192.168.122.1.1.1</param>
+                <!-- read_mode: notification (default, PLC pushes updates) | polling (synchronous SUM read) -->
+                <param name="read_mode">${read_mode}</param>
             </xacro:unless>
         </hardware>
@@ -32,5 +35,7 @@
             <xacro:state_interface_PLC name="statusError" PLC_symbol="MAIN.statusError" PLC_type="BOOL"/>
             <xacro:state_interface_PLC name="batteryVoltage" PLC_symbol="MAIN.batteryVoltage" PLC_type="REAL"/>
-            <xacro:state_interface_PLC name="currentPos_0" PLC_symbol="MAIN.currentPos" PLC_type="LREAL" n_elements="2" index="0" />
+            <!-- currentPos changes every cycle, so stream it cyclically (1 ms) rather than on-change.
+                 The first interface naming MAIN.currentPos sets the notification config for the whole array. -->
+            <xacro:state_interface_PLC name="currentPos_0" PLC_symbol="MAIN.currentPos" PLC_type="LREAL" n_elements="2" index="0" notify_mode="cyclic" notify_cycle_ms="1" />
             <xacro:state_interface_PLC name="currentPos_1" PLC_symbol="MAIN.currentPos" PLC_type="LREAL" n_elements="2" index="1" />
             <xacro:state_interface_PLC name="pickCount" PLC_symbol="MAIN.pickCount" PLC_type="UINT" />
@@ -40,5 +45,5 @@
             <xacro:state_interface_PLC name="joggingEnabled" PLC_symbol="MAIN.joggingEnabled" PLC_type="BOOL" />
             <xacro:state_interface_PLC name="myRobotMode" PLC_symbol="MAIN.myRobotMode" PLC_type="UDINT"/>
-            <xacro:state_interface_PLC name="motionType" PLC_symbol="MAIN.motionType" PLC_type="UDINT"/>
+            <xacro:state_interface_PLC name="motionType" PLC_symbol="MAIN.motionType" PLC_type="USINT"/>
             <xacro:state_interface_PLC name="commandPos_0" PLC_symbol="MAIN.commandPos" PLC_type="BOOL" n_elements="2" index="0" />
             <xacro:state_interface_PLC name="commandPos_1" PLC_symbol="MAIN.commandPos" PLC_type="BOOL" n_elements="2" index="1" />
